File: hardware/kicad/openems_interface_v1/sheets/09_connectors_weact.kicad_sch (KiCad schematic)
At the start: 4 parts, among them J1 1-776180-1, J2 1-770669-1, J3 WeAct_P1_2x25, J4 WeAct_P2_2x25

Commit message: feat(hw): nets J1/J2 no PCB + zones PGND + star GND no sch
Atribui pads AMPSEAL a partir de pinmap_logical.md (autoridade),
adiciona pours PGND F/B, e evita curto de terras no esquemático
(star só via NetTie no layout). Script annotate_pcb_nets.py.
Connections:
- net AGND: no longer J1.14 (Pin_14), J1.17 (Pin_17), J1.18 (Pin_18), J1.30 (Pin_30), J1.33 (Pin_33), J2.19 (Pin_19), J2.20 (Pin_20), J2.21 (Pin_21)
- new net CAN_SHLD: J1.14 (Pin_14), J1.33 (Pin_33)
- new net CMP_GND: J1.17 (Pin_17), J1.18 (Pin_18), J1.30 (Pin_30)
- new net PGND: J2.19 (Pin_19), J2.20 (Pin_20), J2.21 (Pin_21)
Other:
- note added: "STAR = PCB NetTie only"
- note added: "★ STAR GND — unir SÓ no layout (NetTie / ponte copper)\nPGND | SGND | AGND | SHIELD_GND = nets SEPARADAS no esquemático\nNo PCB: um único ponto de união. Correntes INJ/IGN/ETB ≠ SGND/AGND"
- note removed: "STAR"
- note removed: "★ STAR GND — único ponto de união\nPGND + SGND + AGND + SHIELD_GND\nCorrentes INJ/IGN/ETB NUNCA atravessam SGND/AGND"
