File: hardware/openems_ecu/openems_ecu.kicad_pcb (KiCad board)
At the start: 2 copper layers, 80.6 x 93.7 mm, 254 parts, among them J1 USB_B_Mini, J12 Conn_01x01, J13 Conn_01x01, J15 Conn_01x01, J17 Conn_01x01, J19 Conn_01x06, J2 Conn_02x05_Odd_Even, J3 Conn_01x01, J4 Conn_02x05_Counter_Clockwise, J5 Conn_01x01, J6 Micro_SD_Card_Det, J7 TC2030, Q1 IPD30N06S2L-23, SW1 SW_Push, SW2 SW_Push, SW3 SW_Push, SW4 SW_Push, U1 STM32F427VGT6, U10 VNLD5090, U2 TLE8888QK, U3 molex_48pin_MRE, U31 MIC4427, U32 MIC4427, U33 MIC4427, U35 MCP6004, U36 MCP6004, U4 TLE9201SG, U46 MCP6004, U5 LM1117-3.3, U7 XC6206 3.3V, U8 MCP6004, U9 VNLD5090, X1 8MHz 20pF, Y2 32768 Hz

Commit message: feat(hw): STM32H562 sheet, INJEN PE14, and 6-pad PCB rework
H562VGTx LQFP100 does not bond PE1 (pad 98 is VCAP). Move INJEN to PE14
in firmware and docs, replace the MCU sheet with mcu_h562, rework
VCAP/VDDUSB/VSSA copper on the mRE PCB, and wire TLE enables to PE14/PE3.
Parts:
- added C100: 2.2uF, Capacitor_SMD:C_0603_1608Metric, F.Cu at (65.0, 81.3)
- U1: value STM32F427VGT6 -> STM32H562VGT6
- moved C25 22.9 mm to (45.5, 91.3), turned to 180 degrees
Connections:
- C26 pad 1: Net-(C26-Pad1) -> /VDD
- U1 pad 19: /VDD -> GND
- U1 pad 48: /PB11 -> Net-(C100-Pad1)
- U1 pad 49: Net-(C25-Pad1) -> GND
- U1 pad 73: Net-(C26-Pad1) -> /VDD
- U1 pad 98: /PE1 -> Net-(C25-Pad1)
- U2 pad 24: /MCU/PD11 -> /MCU/PE14
- U2 pad 27: /MCU/PD10 -> /PE3
Routing:
- net /PE3: track 10.9 -> 57.9 mm
- net /MCU/PE14: track 23.5 -> 46.2 mm
- net GND: track 111.8 -> 117.8 mm, vias 525 -> 529
- net Net-(C25-Pad1): track 3.75 -> 0.12 mm
- net 264: track 0.00 -> 2.45 mm
- net Net-(C26-Pad1): track 5.04 -> 2.92 mm
- net /MCU/PD10: track 26.3 -> 24.2 mm
- net /PE1: track 9.48 -> 8.24 mm
- net /PB11: track 24.0 -> 22.9 mm
- net /MCU/PD11: track 24.7 -> 24.2 mm
Other:
- board text added: "H562 rework: pad19=VSSA/GND pad48/98=VCAP+2.2uF pad49=VSS/GND pad73=VDDUSB/VDD — see docs/hw/mcu_f407_to_h562_pin_map.md"
