File: hardware/openems_ecu/openems_ecu.kicad_pcb (KiCad board)
At the start: 2 copper layers, 80.6 x 93.7 mm, 255 parts, among them J1 USB_B_Mini, J12 Conn_01x01, J13 Conn_01x01, J15 Conn_01x01, J17 Conn_01x01, J19 Conn_01x06, J2 Conn_02x05_Odd_Even, J3 Conn_01x01, J4 Conn_02x05_Counter_Clockwise, J5 Conn_01x01, J6 Micro_SD_Card_Det, J7 TC2030, Q1 IPD30N06S2L-23, SW1 SW_Push, SW2 SW_Push, SW3 SW_Push, SW4 SW_Push, U1 STM32H562VGT6, U10 VNLD5090, U2 TLE8888QK, U3 molex_48pin_MRE, U31 MIC4427, U32 MIC4427, U33 MIC4427, U35 MCP6004, U36 MCP6004, U4 TLE9201SG, U46 MCP6004, U5 LM1117-3.3, U7 XC6206 3.3V, U8 MCP6004, U9 VNLD5090, X1 8MHz 20pF, Y2 32768 Hz

Commit message: feat(hw): esquemático e PCB alinhados ao pinout VGT6 do TLE8888
Root sheet e a sheet TLE8888-1QK passam a usar nomes de GPIO nos pinos
hierárquicos (PE9, PB12, PA0, …) em vez dos nomes funcionais do mRE,
casando com src/hal/out_pins.h e docs/hw/netlist_v1.md:

  IGN IN5-8   PD12-15 → PE9/11/13/15
  SPI         PD5+PB3/4/5 → PB12-15
  CAN         PB6/PB12 → PB9/PB8
  VROUT       PC6 → PA0
  VVT IN11/12 PE7/8 → PB6/7   (PE7/8 ficam livres para ETB DIR)
  Flash SPI e LIN PD8/9 desligados do MCU

PCB: netlist sincronizado (293 pads), pad C100 com duplo-net do mRE
corrigido, ~567 items de cobre legado removidos e 21 sinais VGT6
U1↔U2 roteados manhattan em F.Cu 0,25 mm.

DRC continua PENDENTE no Pcbnew — as L-tracks podem cruzar outras
redes. Board verificado só quanto a carregar sem crash (a 1ª tentativa
de re-route corrompeu o ficheiro por inserir nets depois do último pad;
esta versão abre, 266 nets, 80,8 x 93,9 mm).

Co-Authored-By: Claude Opus 5 <noreply@anthropic.com>
Parts:
- removed LOGO3: LOGO, rusefi_lib:MRE_QR_code
- C100: footprint Capacitor_SMD:C_0603_1608Metric -> C_0603_1608Metric
- moved C25 22.9 mm to (65.1, 79.4), turned to 90 degrees
- moved C100 22.9 mm to (44.4, 91.3)
Connections:
- C100 pad 1: Net-(C100-Pad1) -> /MCU/VCAP_PE1
- C25 pad 1: Net-(C25-Pad1) -> /MCU/VCAP_PB11
- U1 pad 48: Net-(C100-Pad1) -> /MCU/VCAP_PB11
- U1 pad 98: Net-(C25-Pad1) -> /MCU/VCAP_PE1
- U2 pad 24: /MCU/PE14 -> /MCU/PD11
- U2 pad 27: /PE3 -> /MCU/PD10
Routing:
- net /PE3: track 57.9 -> 10.9 mm
- net /MCU/PE14: track 46.2 -> 23.5 mm
- net /MCU/VCAP_PB11: track 0.00 -> 7.08 mm
- net GND: track 117.8 -> 111.8 mm, vias 529 -> 525
- net /VDD: track 308.7 -> 312.9 mm
- net Net-(C25-Pad1): track 0.12 -> 3.75 mm
- net /MCU/VCAP_PE1: track 0.00 -> 2.77 mm
- net 264: track 2.45 -> 0.00 mm
- net Net-(C26-Pad1): track 2.92 -> 5.04 mm
- net /MCU/PD10: track 24.2 -> 26.3 mm
- net /PE1: track 8.24 -> 9.48 mm
- net /PB11: track 22.9 -> 24.0 mm
- net /MCU/PD11: track 24.2 -> 24.7 mm
Other:
- board text added: "OpenEMS"
- board text added: "OpenEMS / H562 R0.1 PCB DESIGN BY OLA RUUD R0.2 PCB DESIGN BY DAECU R0.3 PCB DESIGN BY DAECU R0.4 PCB DESIGN BY DBECKER R0.5 PCB DESIGN BY COMMUNITY"
- board text added: "OpenEMS H562"
- board text added: "STM32H562VG"
- board text removed: "H562 rework: pad19=VSSA/GND pad48/98=VCAP+2.2uF pad49=VSS/GND pad73=VDDUSB/VDD — see docs/hw/mcu_f407_to_h562_pin_map.md"
- board text removed: "R0.1 PCB DESIGN BY OLA RUUD R0.2 PCB DESIGN BY DAECU R0.3 PCB DESIGN BY DAECU R0.4 PCB DESIGN BY DBECKER R0.5 PCB DESIGN BY COMMUNITY"
- board text removed: "RUSEFI.COM"
- board text removed: "STM32F407VG"
- board text removed: "microRusEFI R0.6.0"
- board text removed: "rusefi.com/s/microrusefi"
