File: hardware/openems_ecu/openems_ecu.kicad_sch (KiCad schematic)
At the start: 57 parts, among them J12 Conn_01x01, J13 Conn_01x01, J3 Conn_01x01, J4 Conn_02x05_Counter_Clockwise, J5 Conn_01x01, U3 molex_48pin_MRE, U7 XC6206 3.3V

Commit message: feat(hw): STM32H562 sheet, INJEN PE14, and 6-pad PCB rework
H562VGTx LQFP100 does not bond PE1 (pad 98 is VCAP). Move INJEN to PE14
in firmware and docs, replace the MCU sheet with mcu_h562, rework
VCAP/VDDUSB/VSSA copper on the mRE PCB, and wire TLE enables to PE14/PE3.
Connections:
- net PB11: no longer names the net of U3.J12
- net PE1 renamed PE14
Other:
- sheet MCU: file stm32.kicad_sch -> mcu_h562.kicad_sch
- sheet MCU ports: added none; removed PB11, PE1
- note added: "OpenEMS: INJEN=PE14, IGNEN=PE3 (TLE enables). Status LEDs reassigned — PE1 not bonded on H562 LQFP100."
- note removed: "PE1 is yellow- warning PE2 is blue - communication PE3 is red - fatal PE4 is green - running"
Changed lines of the file:
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@@
 	(wire
 		(pts
-			(xy 201.93 156.845) (xy 203.835 156.845)
-		)
-		(stroke
-			(width 0)
-			(type default)
-		)
-	)
-	(wire
-		(pts
 			(xy 340.36 54.61) (xy 341.63 54.61)
 		)
@@
 		)
 	)
-	(text "PE1 is yellow- warning\nPE2 is blue - communication\nPE3 is red - fatal\nPE4 is green - running"
+	(text "OpenEMS: INJEN=PE14, IGNEN=PE3 (TLE enables).\nStatus LEDs reassigned — PE1 not bonded on H562 LQFP100."
 		(exclude_from_sim no)
 		(at 372.11 157.48 0)
@@
 		)
 	)
-	(label "PB11"
-		(at 169.545 203.835 180)
-		(effects
-			(font
-				(size 1.27 1.27)
-			)
-			(justify right bottom)
-		)
-	)
 	(label "5V1"
 		(at 228.6 147.955 180)
@@
 		)
 	)
-	(label "PE1"
-		(at 203.835 156.845 0)
+	(label "PE14"
+		(at 203.835 97.155 0)
 		(effects
 			(font
@@
 		)
 	)
-	(label "PE1"
+	(label "PE14"
 		(at 346.71 148.59 180)
 		(effects
@@
 			)
 		)
-		(property "Sheetfile" "stm32.kicad_sch"
+		(property "Sheetfile" "mcu_h562.kicad_sch"
 			(at 170.18 244.4246 0)
 			(effects
@@
 			)
 		)
-		(pin "PB11" input
-			(at 170.18 203.835 180)
-			(effects
-				(font
-					(size 1.524 1.524)
-				)
-				(justify left)
-			)
-		)
 		(pin "PB13" input
 			(at 170.18 193.04 180)
@@
 			)
 		)
-		(pin "PE1" input
-			(at 201.93 156.845 0)
-			(effects
-				(font
-					(size 1.524 1.524)
-				)
-				(justify right)
-			)
-		)
 		(pin "PB9" input
 			(at 201.93 224.155 0)
@@
 		)
 	)
+	(wire
+		(pts
+			(xy 201.93 97.155) (xy 203.835 97.155)
+		)
+		(stroke
+			(width 0)
+			(type default)
+		)
+	)
+	(label "PE14"
+		(at 230.0 186.055 0)
+		(effects
+			(font
+				(size 1.27 1.27)
+				(thickness 0.254)
+				(bold yes)
+			)
+			(justify left bottom)
+		)
+	)
+	(label "PE3"
+		(at 230.0 183.515 0)
+		(effects
+			(font
+				(size 1.27 1.27)
+				(thickness 0.254)
+				(bold yes)
+			)
+			(justify left bottom)
+		)
+	)
+	(wire
+		(pts
+			(xy 228.6 186.055) (xy 230.0 186.055)
+		)
+		(stroke
+			(width 0)
+			(type default)
+		)
+	)
+	(wire
+		(pts
+			(xy 228.6 183.515) (xy 230.0 183.515)
+		)
+		(stroke
+			(width 0)
+			(type default)
+		)
+	)
