File: hardware/openems_ecu/openems_ecu.kicad_sch (KiCad schematic)
At the start: 57 parts, among them J12 Conn_01x01, J13 Conn_01x01, J3 Conn_01x01, J4 Conn_02x05_Counter_Clockwise, J5 Conn_01x01, U3 molex_48pin_MRE, U7 XC6206 3.3V

Commit message: feat(hw): esquemático e PCB alinhados ao pinout VGT6 do TLE8888
Root sheet e a sheet TLE8888-1QK passam a usar nomes de GPIO nos pinos
hierárquicos (PE9, PB12, PA0, …) em vez dos nomes funcionais do mRE,
casando com src/hal/out_pins.h e docs/hw/netlist_v1.md:

  IGN IN5-8   PD12-15 → PE9/11/13/15
  SPI         PD5+PB3/4/5 → PB12-15
  CAN         PB6/PB12 → PB9/PB8
  VROUT       PC6 → PA0
  VVT IN11/12 PE7/8 → PB6/7   (PE7/8 ficam livres para ETB DIR)
  Flash SPI e LIN PD8/9 desligados do MCU

PCB: netlist sincronizado (293 pads), pad C100 com duplo-net do mRE
corrigido, ~567 items de cobre legado removidos e 21 sinais VGT6
U1↔U2 roteados manhattan em F.Cu 0,25 mm.

DRC continua PENDENTE no Pcbnew — as L-tracks podem cruzar outras
redes. Board verificado só quanto a carregar sem crash (a 1ª tentativa
de re-route corrompeu o ficheiro por inserir nets depois do último pad;
esta versão abre, 266 nets, 80,8 x 93,9 mm).

Co-Authored-By: Claude Opus 5 <noreply@anthropic.com>
Connections:
- net CRANK: no longer D28.2 (A)
- net MCU/PB7 renamed PB7
- net MCU/PE6 renamed PE6
- net TLE8888-1QK/IGN_OUT_1 renamed TLE8888-1QK/IGN1
- net TLE8888-1QK/IGN_OUT_2 renamed TLE8888-1QK/IGN2
- net TLE8888-1QK/IGN_OUT_3 renamed TLE8888-1QK/IGN3
- net TLE8888-1QK/IGN_OUT_4 renamed TLE8888-1QK/IGN4
Other:
- sheet TLE8888-1QK ports: added IGN1, IGN2, IGN3, IGN4, INJ1, INJ2, INJ3, INJ4, PA0, PB12, PB13, PB14, PB15, PB6, PB7, PB8, PB9, PE0, PE10, PE11, PE12, PE13, PE14, PE15, PE2, PE3, PE4, PE6, PE9; removed CAN_RX, CAN_TX, CRNK_IN, CSN, FCLP, IGN_EN, IGN_IN_1, IGN_IN_2, IGN_IN_3, IGN_IN_4, IGN_OUT_1, IGN_OUT_2, IGN_OUT_3, IGN_OUT_4, INJ_1, INJ_2, INJ_3, INJ_4, INJ_EN, INJ_IN_1, INJ_IN_2, INJ_IN_3, INJ_IN_4, IN_10, IN_11, IN_12, IN_9, SDO, SIP
- note added: "OpenEMS VGT6: TLE sheet pins = MCU GPIO names. INJ PE0/2/4/6 IGN PE9/11/13/15 EN PE14/PE3. PUMP/FAN PE10/12 VVT PB6/7 SPI PB12-15 CAN PB8/9 CKP PA0. Outs IGN1-4/INJ1-4. Strap SIN=GND FCLN=VDDIO."
- note removed: "OpenEMS: INJEN=PE14, IGNEN=PE3 (TLE enables). Status LEDs reassigned — PE1 not bonded on H562 LQFP100."
