File: hardware/openems_ecu/TLE8888-1QK.kicad_sch (KiCad schematic)
At the start: 40 parts, among them J15 Conn_01x01, J17 Conn_01x01, Q1 IPD30N06S2L-23, U2 TLE8888QK

Commit message: feat(hw): esquemático e PCB alinhados ao pinout VGT6 do TLE8888
Root sheet e a sheet TLE8888-1QK passam a usar nomes de GPIO nos pinos
hierárquicos (PE9, PB12, PA0, …) em vez dos nomes funcionais do mRE,
casando com src/hal/out_pins.h e docs/hw/netlist_v1.md:

  IGN IN5-8   PD12-15 → PE9/11/13/15
  SPI         PD5+PB3/4/5 → PB12-15
  CAN         PB6/PB12 → PB9/PB8
  VROUT       PC6 → PA0
  VVT IN11/12 PE7/8 → PB6/7   (PE7/8 ficam livres para ETB DIR)
  Flash SPI e LIN PD8/9 desligados do MCU

PCB: netlist sincronizado (293 pads), pad C100 com duplo-net do mRE
corrigido, ~567 items de cobre legado removidos e 21 sinais VGT6
U1↔U2 roteados manhattan em F.Cu 0,25 mm.

DRC continua PENDENTE no Pcbnew — as L-tracks podem cruzar outras
redes. Board verificado só quanto a carregar sem crash (a 1ª tentativa
de re-route corrompeu o ficheiro por inserir nets depois do último pad;
esta versão abre, 266 nets, 80,8 x 93,9 mm).

Co-Authored-By: Claude Opus 5 <noreply@anthropic.com>
Connections:
- net CAN_RX renamed PB8
- net CAN_TX renamed PB9
- net CRNK_IN renamed PA0
- net CSN renamed PB12
- net FCLP renamed PB13
- net IGN_EN renamed PE3
- net IGN_IN_1 renamed PE9
- net IGN_IN_2 renamed PE11
- net IGN_IN_3 renamed PE13
- net IGN_IN_4 renamed PE15
- net IGN_OUT_1 renamed IGN1
- net IGN_OUT_2 renamed IGN2
- net IGN_OUT_3 renamed IGN3
- net IGN_OUT_4 renamed IGN4
- net INJ_1 renamed INJ1
- net INJ_2 renamed INJ2
- net INJ_3 renamed INJ3
- net INJ_4 renamed INJ4
- net INJ_EN renamed PE14
- net INJ_IN_1 renamed PE0
- net INJ_IN_2 renamed PE2
- net INJ_IN_3 renamed PE4
- net INJ_IN_4 renamed PE6
- net IN_10 renamed PE12
- net IN_11 renamed PB6
- net IN_12 renamed PB7
- net IN_9 renamed PE10
- net SDO renamed PB14
- net SIP renamed PB15
Changed lines of the file:
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@@
 		)
 	)
-	(hierarchical_label "IGN_IN_2"
+	(hierarchical_label "PE11"
 		(shape input)
 		(at 294.64 227.33 0)
@@
 		)
 	)
-	(hierarchical_label "IGN_OUT_3"
+	(hierarchical_label "IGN3"
 		(shape input)
 		(at 203.2 238.76 180)
@@
 		)
 	)
-	(hierarchical_label "SIP"
+	(hierarchical_label "PB15"
 		(shape input)
 		(at 227.33 259.08 270)
@@
 		)
 	)
-	(hierarchical_label "INJ_EN"
+	(hierarchical_label "PE14"
 		(shape input)
 		(at 313.69 261.62 0)
@@
 		)
 	)
-	(hierarchical_label "IGN_OUT_2"
+	(hierarchical_label "IGN2"
 		(shape input)
 		(at 203.2 236.22 180)
@@
 		)
 	)
-	(hierarchical_label "IGN_EN"
+	(hierarchical_label "PE3"
 		(shape input)
 		(at 313.69 242.57 0)
@@
 		)
 	)
-	(hierarchical_label "IGN_IN_1"
+	(hierarchical_label "PE9"
 		(shape input)
 		(at 294.64 229.87 0)
@@
 		)
 	)
-	(hierarchical_label "IGN_IN_4"
+	(hierarchical_label "PE15"
 		(shape input)
 		(at 294.64 222.25 0)
@@
 		)
 	)
-	(hierarchical_label "INJ_2"
+	(hierarchical_label "INJ2"
 		(shape input)
 		(at 254 167.64 90)
@@
 		)
 	)
-	(hierarchical_label "CAN_RX"
+	(hierarchical_label "PB8"
 		(shape input)
 		(at 294.64 201.93 0)
@@
 		)
 	)
-	(hierarchical_label "INJ_1"
+	(hierarchical_label "INJ1"
 		(shape input)
 		(at 259.08 167.64 90)
@@
 		)
 	)
-	(hierarchical_label "INJ_IN_1"
+	(hierarchical_label "PE0"
 		(shape input)
 		(at 294.64 240.03 0)
@@
 		)
 	)
-	(hierarchical_label "IN_11"
+	(hierarchical_label "PB6"
 		(shape input)
 		(at 294.64 214.63 0)
@@
 		)
 	)
-	(hierarchical_label "INJ_4"
+	(hierarchical_label "INJ4"
 		(shape input)
 		(at 243.84 167.64 90)
@@
 		)
 	)
-	(hierarchical_label "IGN_IN_3"
+	(hierarchical_label "PE13"
 		(shape input)
 		(at 294.64 224.79 0)
@@
 		)
 	)
-	(hierarchical_label "FCLP"
+	(hierarchical_label "PB13"
 		(shape input)
 		(at 232.41 259.08 270)
@@
 		)
 	)
-	(hierarchical_label "IN_12"
+	(hierarchical_label "PB7"
 		(shape input)
 		(at 294.64 212.09 0)
@@
 		)
 	)
-	(hierarchical_label "INJ_IN_3"
+	(hierarchical_label "PE4"
 		(shape input)
 		(at 294.64 234.95 0)
@@
 		)
 	)
-	(hierarchical_label "INJ_3"
+	(hierarchical_label "INJ3"
 		(shape input)
 		(at 248.92 167.64 90)
@@
 		)
 	)
-	(hierarchical_label "IGN_OUT_4"
+	(hierarchical_label "IGN4"
 		(shape input)
 		(at 203.2 241.3 180)
@@
 		)
 	)
-	(hierarchical_label "SDO"
+	(hierarchical_label "PB14"
 		(shape input)
 		(at 224.79 259.08 270)
@@
 		)
 	)
-	(hierarchical_label "INJ_IN_4"
+	(hierarchical_label "PE6"
 		(shape input)
 		(at 294.64 232.41 0)
@@
 		)
 	)
-	(hierarchical_label "IN_10"
+	(hierarchical_label "PE12"
 		(shape input)
 		(at 294.64 217.17 0)
@@
 		)
 	)
-	(hierarchical_label "CSN"
+	(hierarchical_label "PB12"
 		(shape input)
 		(at 222.25 259.08 270)
@@
 		)
 	)
-	(hierarchical_label "CAN_TX"
+	(hierarchical_label "PB9"
 		(shape input)
 		(at 294.64 199.39 0)
@@
 		)
 	)
-	(hierarchical_label "CRNK_IN"
+	(hierarchical_label "PA0"
 		(shape input)
 		(at 269.24 269.24 0)
@@
 		)
 	)
-	(hierarchical_label "IGN_OUT_1"
+	(hierarchical_label "IGN1"
 		(shape input)
 		(at 203.2 233.68 180)
@@
 		)
 	)
-	(hierarchical_label "INJ_IN_2"
+	(hierarchical_label "PE2"
 		(shape input)
 		(at 294.64 237.49 0)
@@
 		)
 	)
-	(hierarchical_label "IN_9"
+	(hierarchical_label "PE10"
 		(shape input)
 		(at 294.64 219.71 0)
