File: hardware/openems_v1/openems_v1.kicad_pcb (KiCad board)
At the start: 4 copper layers, 160 x 110 mm, 0 parts

Commit message: feat(hw): fecha esquemático v2 — sheets 01/02/03/05/07/11 desenhadas, ERC 0
- 01_power: nova — P-FET reverse (Q1) + F1 30A + SMBJ24CA + bulk 100µF/100nF,
  star GND (PGND/SGND/AGND) via PWR_FLAG na sheet produtora, VBAT limpo para
  o resto da placa (buck/LDO ficam no TPS65381A, sheet PMIC)
- 02_ckp / 03_cmp: CKP Hall (espelho do CMP) → MCU.PA0/PA1
- 05_analog: refeita do zero a partir do pinout_v2 (13 canais ADC), mapa
  pré-v2 descartado
- 11_mcu_h562: netlist U1 corrigido (lib_id não resolvia pinos — 100 pinos
  caíam na mesma net); globals PA0/PA1/PB4 sincronizados com as sheets acima
- 07_flex: pino corrigido para PB4 (pinout_v2)
- READMEs (hardware/openems_v1, docs/hw/schematic) actualizados ao estado
  real por sheet

Passos 1-5 do roadmap do esquemático fechados; ERC isolado por sheet em 0
erros (avisos residuais são globals sem sheet destino ainda — esperado).

Co-Authored-By: Claude Sonnet 5 <noreply@anthropic.com>
Changed lines of the file:
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@@
 		(end 23 20)
 		(stroke
-			(width 0)
+			(width 0.1)
 			(type default)
 		)
@@
 		(end 20 23)
 		(stroke
-			(width 0)
+			(width 0.1)
 			(type default)
 		)
@@
 		(end 177 20)
 		(stroke
-			(width 0)
+			(width 0.1)
 			(type default)
 		)
@@
 		(end 20 127)
 		(stroke
-			(width 0)
+			(width 0.1)
 			(type default)
 		)
@@
 		(end 180 23)
 		(stroke
-			(width 0)
+			(width 0.1)
 			(type default)
 		)
@@
 		(end 23 130)
 		(stroke
-			(width 0)
+			(width 0.1)
 			(type default)
 		)
@@
 		(end 180 127)
 		(stroke
-			(width 0)
+			(width 0.1)
 			(type default)
 		)
@@
 		(end 177 130)
 		(stroke
-			(width 0)
+			(width 0.1)
 			(type default)
 		)
