File: hardware/openems_v1/sheets/11_mcu_h562.kicad_sch (KiCad schematic)
At the start: 0 parts

Commit message: feat(hw): fecha esquemático v2 — sheets 01/02/03/05/07/11 desenhadas, ERC 0
- 01_power: nova — P-FET reverse (Q1) + F1 30A + SMBJ24CA + bulk 100µF/100nF,
  star GND (PGND/SGND/AGND) via PWR_FLAG na sheet produtora, VBAT limpo para
  o resto da placa (buck/LDO ficam no TPS65381A, sheet PMIC)
- 02_ckp / 03_cmp: CKP Hall (espelho do CMP) → MCU.PA0/PA1
- 05_analog: refeita do zero a partir do pinout_v2 (13 canais ADC), mapa
  pré-v2 descartado
- 11_mcu_h562: netlist U1 corrigido (lib_id não resolvia pinos — 100 pinos
  caíam na mesma net); globals PA0/PA1/PB4 sincronizados com as sheets acima
- 07_flex: pino corrigido para PB4 (pinout_v2)
- READMEs (hardware/openems_v1, docs/hw/schematic) actualizados ao estado
  real por sheet

Passos 1-5 do roadmap do esquemático fechados; ERC isolado por sheet em 0
erros (avisos residuais são globals sem sheet destino ainda — esperado).

Co-Authored-By: Claude Sonnet 5 <noreply@anthropic.com>
Parts:
- added C1, C10, C11, C2, C3, C4, C5, C9: 100nF, Capacitor_SMD:C_0603_1608Metric, symbol Device:C
- added C12, C13: 12pF, Capacitor_SMD:C_0402_1005Metric, symbol Device:C
- added C6: 1uF, Capacitor_SMD:C_0805_2012Metric, symbol Device:C
- added C7, C8: 2.2uF, Capacitor_SMD:C_0805_2012Metric, symbol Device:C
- added J1: Conn_ARM_SWD_TagConnect_TC2030-NL, Connector:Tag-Connect_TC2030-IDC-NL_2x03_P1.27mm_Vertical, symbol Connector:Conn_ARM_SWD_TagConnect_TC2030-NL
- added JP1: BOOT0_DFU, Connector_PinHeader_2.54mm:PinHeader_1x02_P2.54mm_Vertical, symbol Connector_Generic:Conn_01x02
- added R1: 10k, Resistor_SMD:R_0603_1608Metric, symbol Device:R
- added SW1: NRST, Button_Switch_SMD:SW_SPST_PTS810, symbol Switch:SW_Push
- added U1: STM32H562VGTx, Package_QFP:LQFP-100_14x14mm_P0.5mm, symbol STM32H562VGTx
- added X1: 3225-8.00-10-10-10/A, Crystal:Crystal_SMD_3225-4Pin_3.2x2.5mm, symbol Device:Crystal_GND24
- added Y2: 32.768kHz DNP, Crystal:Crystal_SMD_3215-2Pin_3.2x1.5mm, symbol Device:Crystal
Connections:
- new net +3V3: C1.1, C10.1, C2.1, C3.1, C4.1, C5.1, C6.1, C9.1, J1.1 (VCC), JP1.2 (Pin_2), U1.100 (VDD), U1.11 (VDD), U1.28 (VDD), U1.50 (VDD), U1.6 (VBAT), U1.73 (VDDUSB), U1.75 (VDD)
- new net AGND: U1.19 (VSSA), U1.20 (VREF-)
- new net GND: C1.2, C10.2, C11.2, C12.2, C13.2, C2.2, C3.2, C4.2, C5.2, C6.2, C7.2, C8.2, C9.2, J1.5 (GND), R1.2, SW1.2, U1.10 (VSS), U1.27 (VSS), U1.49 (VSS), U1.74 (VSS), U1.99 (VSS), X1.2, X1.4
- new net MCU.BOOT0: JP1.1 (Pin_1), R1.1, U1.94 (BOOT0)
- new net MCU.NRST: C11.1, J1.3 (~{RESET}), SW1.1, U1.14 (NRST)
- new net MCU.OSC_IN: C12.1, U1.12 (PH0), X1.1
- new net MCU.OSC_OUT: C13.1, U1.13 (PH1), X1.3
- new net MCU.PA0: U1.23 (PA0)
- new net MCU.PA1: U1.24 (PA1)
- new net MCU.PA13: J1.2 (SWDIO), U1.72 (PA13(JTMS)
- new net MCU.PA14: J1.4 (SWCLK), U1.76 (PA14(JTCK)
- new net MCU.PA2: U1.25 (PA2)
- new net MCU.PA3: U1.26 (PA3)
- new net MCU.PA4: U1.29 (PA4)
- new net MCU.PA5: U1.30 (PA5)
- new net MCU.PA7: U1.32 (PA7)
- new net MCU.PB0: U1.35 (PB0)
- new net MCU.PB1: U1.36 (PB1)
- new net MCU.PB4: U1.90 (PB4(NJTRST))
- new net MCU.PC0: U1.15 (PC0)
- new net MCU.PC1: U1.16 (PC1)
- new net MCU.PC2: U1.17 (PC2)
- new net MCU.PC3: U1.18 (PC3)
- new net MCU.PC4: U1.33 (PC4)
- new net MCU.PC5: U1.34 (PC5)
- new net MCU.VCAP1: C7.1, U1.48 (VCAP)
- new net MCU.VCAP2: C8.1, U1.98 (VCAP)
- new net VDDA: U1.21 (VREF+), U1.22 (VDDA)
- no-connect marks 0 -> 7
Changed lines of the file:
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@@
 (kicad_sch
-	(version 20260101)
+	(version 20260306)
 	(generator "eeschema")
 	(generator_version "10.0")
 	(paper "A4")
-	(sheet_instances
-		(path "/"
-			(page "1")
-		)
-	)
-)
