File: hardware/openems_v1/sheets/05_analog.kicad_sch (KiCad schematic)
At the start: 0 parts

Commit message: feat(hw): fecha esquemático v2 — sheets 01/02/03/05/07/11 desenhadas, ERC 0
- 01_power: nova — P-FET reverse (Q1) + F1 30A + SMBJ24CA + bulk 100µF/100nF,
  star GND (PGND/SGND/AGND) via PWR_FLAG na sheet produtora, VBAT limpo para
  o resto da placa (buck/LDO ficam no TPS65381A, sheet PMIC)
- 02_ckp / 03_cmp: CKP Hall (espelho do CMP) → MCU.PA0/PA1
- 05_analog: refeita do zero a partir do pinout_v2 (13 canais ADC), mapa
  pré-v2 descartado
- 11_mcu_h562: netlist U1 corrigido (lib_id não resolvia pinos — 100 pinos
  caíam na mesma net); globals PA0/PA1/PB4 sincronizados com as sheets acima
- 07_flex: pino corrigido para PB4 (pinout_v2)
- READMEs (hardware/openems_v1, docs/hw/schematic) actualizados ao estado
  real por sheet

Passos 1-5 do roadmap do esquemático fechados; ERC isolado por sheet em 0
erros (avisos residuais são globals sem sheet destino ainda — esperado).

Co-Authored-By: Claude Sonnet 5 <noreply@anthropic.com>
Parts:
- added C20, C21, C22, C23, C24, C25, C26, C27, C28, C29, C31, C32: 100nF, Capacitor_SMD:C_0603_1608Metric, symbol Device:C
- added C30: 1uF, Capacitor_SMD:C_0805_2012Metric, symbol Device:C
- added D10, D11, D12, D13, D14, D15, D16, D17, D18, D19, D20, D21: 3V3, Diode_SMD:D_SOD-323, symbol Device:D_TVS
- added R100, R103, R108, R111, R114, R117, R120, R123, R127: 10k, Resistor_SMD:R_0603_1608Metric, symbol Device:R
- added R101, R104, R109, R112, R115, R118, R121, R124: 15k, Resistor_SMD:R_0603_1608Metric, symbol Device:R
- added R102, R105, R106, R107, R110, R113, R116, R119, R122, R125, R128, R130, R132: 1k, Resistor_SMD:R_0603_1608Metric, symbol Device:R
- added R126: 47k, Resistor_SMD:R_0603_1608Metric, symbol Device:R
- added R129, R131: 2k49, Resistor_SMD:R_0603_1608Metric, symbol Device:R
Connections:
- new net +5V_SENS_A: R129.1, R131.1
- new net AGND: C20.2, C21.2, C22.2, C23.2, C24.2, C25.2, C26.2, C27.2, C28.2, C29.2, C30.2, C31.2, C32.2, D10.2 (A2), D11.2 (A2), D12.2 (A2), D13.2 (A2), D14.2 (A2), D15.2 (A2), D16.2 (A2), D17.2 (A2), D18.2 (A2), D19.2 (A2), D20.2 (A2), D21.2 (A2)
- new net J1.APP1_SIG: R111.1
- new net J1.APP2_SIG: R114.1
- new net J1.CLT_SIG: D20.1 (A1), R129.2, R130.1
- new net J1.ETB_TPS2_SIG: R120.1
- new net J1.EWG_POS_SIG: R108.1
- new net J1.FUEL_P_SIG: R103.1
- new net J1.IAT_SIG: D21.1 (A1), R131.2, R132.1
- new net J1.MAP_SIG: R123.1
- new net J1.OIL_P_SIG: R100.1
- new net J1.TPS1_SIG: R117.1
- new net MCU.PA2: C20.1, R102.2
- new net MCU.PA3: C21.1, R105.2
- new net MCU.PA4: C22.1, D12.1 (A1), R106.2
- new net MCU.PA5: C23.1, D13.1 (A1), R107.2
- new net MCU.PA7: C24.1, R110.2
- new net MCU.PB0: C25.1, R113.2
- new net MCU.PB1: C26.1, R116.2
- new net MCU.PC0: C27.1, R119.2
- new net MCU.PC1: C28.1, R122.2
- new net MCU.PC2: C29.1, R125.2
- new net MCU.PC3: C30.1, R128.2
- new net MCU.PC4: C31.1, R130.2
- new net MCU.PC5: C32.1, R132.2
- new net N_APP1_DIV: D15.1 (A1), R111.2, R112.1, R113.1
- new net N_APP2_DIV: D16.1 (A1), R114.2, R115.1, R116.1
- new net N_ETB2_DIV: D18.1 (A1), R120.2, R121.1, R122.1
- new net N_EWG_DIV: D14.1 (A1), R108.2, R109.1, R110.1
- new net N_FUEL_DIV: D11.1 (A1), R103.2, R104.1, R105.1
- new net N_LAMBDA_UA: R106.1
- new net N_LAMBDA_UR: R107.1
- new net N_MAP_DIV: D19.1 (A1), R123.2, R124.1, R125.1
- new net N_OIL_DIV: D10.1 (A1), R100.2, R101.1, R102.1
- new net N_TPS1_DIV: D17.1 (A1), R117.2, R118.1, R119.1
- new net N_VBATT_DIV: R126.2, R127.1, R128.1
- new net PGND: R127.2
- new net SGND: R101.2, R104.2, R109.2, R112.2, R115.2, R118.2, R121.2, R124.2
- new net VBAT: R126.1
Other:
- note added: "Sheet 05 — ADC pinout_v2 | 13 ch pinout_v2 | OpenEMS v2"
